Commit message: sim stuff

File: src/simulation/urdf/board_arm.urdf.xacro (robot description, xacro)
@@ -1,8 +1,45 @@
 <?xml version="1.1"?>
 <robot xmlns:xacro="http://www.ros.org/wiki/xacro" name="board_arm">
-    <xacro:property name="link_length" value="${5*sqrt(2)/2 - cylinder_radius}"/>
-    <xacro:property name="link_width" value="0.5"/>
-    <xacro:property name="link_height" value="0.5"/>
+    <xacro:property name="tile_size" value="0.25"/>
+    <xacro:property name="link_length" value="${tile_size * 5 * sqrt(2) / 2 - cylinder_radius}"/>
+    <xacro:property name="link_width" value="0.1"/>
+    <xacro:property name="link_height" value="0.1"/>
     <xacro:property name="cylinder_radius" value="${link_width / 2}"/>
+    <xacro:property name="link_mass" value="0.1"/>
+    <gazebo>
+        <plugin name="gazebo_ros_control" filename="libgazebo_ros_control.so">
+            <robotNamespace>/board_arm</robotNamespace>
+        </plugin>
+    </gazebo>
+    <gazebo reference="link1">
+        <material>Gazebo/Black</material>
+    </gazebo>
+    <gazebo reference="link2">
+        <material>Gazebo/Red</material>
+    </gazebo>
+    <gazebo reference="link3">
+        <material>Gazebo/Black</material>
+    </gazebo>
+    <gazebo reference="link4">
+        <material>Gazebo/Red</material>
+    </gazebo>
+    <transmission name="tran1">
+        <type>transmission_interface/SimpleTransmission</type>
+        <joint name="joint1">
+            <hardwareInterface>hardware_interface/EffortJointInterface</hardwareInterface>
+        </joint>
+        <actuator name="motor1">
+            <hardwareInterface>hardware_interface/EffortJointInterface</hardwareInterface>
+        </actuator>
+    </transmission>
+    <transmission name="tran2">
+        <type>transmission_interface/SimpleTransmission</type>
+        <joint name="joint2">
+            <hardwareInterface>hardware_interface/EffortJointInterface</hardwareInterface>
+        </joint>
+        <actuator name="motor2">
+            <hardwareInterface>hardware_interface/EffortJointInterface</hardwareInterface>
+        </actuator>
+    </transmission>
     <material name="Red">
         <color rgba="${220/255} ${0/255} ${25/255} 0.5"/>
@@ -11,9 +48,21 @@
         <color rgba="0.0 0.0 0.0 0.5"/>
     </material>
-    <!-- link0 is the ground or base_link: unmoving -->
-    <link name="link0"/>
+    <!-- world (link0) is the ground or base_link: unmoving -->
+    <link name="world"/>
     <link name="link1">
+        <inertial>
+            <origin xyz="0 0 ${link_height / 2}"/>
+            <mass value="${link_mass}"/>
+            <!--
+            These values are from the inertia matrices from:
+            https://en.wikipedia.org/wiki/List_of_moments_of_inertia#List_of_3D_inertia_tensors
+            -->
+            <inertia
+              ixx="${1/12 * link_mass * (3 * cylinder_radius ** 2 + link_height ** 2)}" ixy="0" ixz="0"
+              iyy="${1/12 * link_mass * (3 * cylinder_radius ** 2 + link_height ** 2)}" iyz="0"
+              izz="${1/2 * link_mass * cylinder_radius ** 2}"/>
+         </inertial>
         <visual name="joint">
-            <origin xyz="0 0 0"/>
+            <origin xyz="0 0 ${link_height / 2}"/>
             <geometry>
                 <cylinder length="${link_height}" radius="${cylinder_radius}"/>
@@ -21,7 +70,23 @@
             <material name="Black"/>
         </visual>
+        <collision name="joint">
+            <origin xyz="0 0 ${link_height / 2}"/>
+            <geometry>
+                <cylinder length="${link_height}" radius="${cylinder_radius}"/>
+            </geometry>
+        </collision>
+    </link>
+    <link name="link2">
+        <inertial>
+            <origin xyz="${link_length / 2 + cylinder_radius} 0 ${link_height / 2}"/>
+            <mass value="${link_mass}"/>
+            <inertia
+              ixx="${1/12 * link_mass * (link_height**2 + link_width**2)}" ixy="0" ixz="0"
+              iyy="${1/12 * link_mass * (link_length**2 + link_height**2)}" iyz="0"
+              izz="${1/12 * link_mass * (link_length**2 + link_width**2)}"/>
+        </inertial>
         <visual name="link">
-            <!-- the "link_length + 2" is there since the frame is in the center of the box -->
-            <origin xyz="${link_length / 2 + cylinder_radius} 0 0"/>
+            <!-- the "link_length / 2" is there since the frame is in the center of the box -->
+            <origin xyz="${link_length / 2 + cylinder_radius} 0 ${link_height / 2}"/>
             <geometry>
                 <box size="${link_length} ${link_width} ${link_height}"/>
@@ -29,8 +94,26 @@
             <material name="Red"/>
         </visual>
+        <collision name="link">
+            <origin xyz="${link_length / 2 + cylinder_radius} 0 ${link_height / 2}"/>
+            <geometry>
+                <box size="${link_length} ${link_width} ${link_height}"/>
+            </geometry>
+        </collision>
     </link>
-    <link name="link2">
+    <link name="link3">
+        <inertial>
+            <origin xyz="0 0 ${link_height / 2}"/>
+            <mass value="${link_mass}"/>
+            <!--
+            These values are from the inertia matrices from:
+            https://en.wikipedia.org/wiki/List_of_moments_of_inertia#List_of_3D_inertia_tensors
+            -->
+            <inertia
+              ixx="${1/12 * link_mass * (3 * cylinder_radius ** 2 + link_height ** 2)}" ixy="0" ixz="0"
+              iyy="${1/12 * link_mass * (3 * cylinder_radius ** 2 + link_height ** 2)}" iyz="0"
+              izz="${1/2 * link_mass * cylinder_radius ** 2}"/>
+        </inertial>
         <visual name="joint">
-            <origin xyz="0 0 0"/>
+            <origin xyz="0 0 ${link_height / 2}"/>
             <geometry>
                 <cylinder length="${link_height}" radius="${cylinder_radius}"/>
@@ -38,6 +121,21 @@
             <material name="Black"/>
         </visual>
+        <collision name="joint">
+            <origin xyz="0 0 ${link_height / 2}"/>
+            <geometry>
+                <cylinder length="${link_height}" radius="${cylinder_radius}"/>
+            </geometry>
+        </collision>
+    </link>
+    <link name="link4">
+        <inertial>
+            <origin xyz="${link_length / 2 + cylinder_radius} 0 ${link_height / 2}"/>
+            <mass value="${link_mass}"/>
+            <inertia ixx="${1/12 * link_mass * (link_height**2 + link_width**2)}" ixy="0" ixz="0"
+                     iyy="${1/12 * link_mass * (link_length**2 + link_height**2)}" iyz="0"
+                     izz="${1/12 * link_mass * (link_length**2 + link_width**2)}"/>
+        </inertial>
         <visual name="link">
-            <origin xyz="${link_length / 2 + cylinder_radius} 0 0"/>
+            <origin xyz="${link_length / 2 + cylinder_radius} 0 ${link_height / 2}"/>
             <geometry>
                 <box size="${link_length} ${link_width} ${link_height}"/>
@@ -45,16 +143,33 @@
             <material name="Red"/>
         </visual>
+        <collision name="link">
+            <origin xyz="${link_length / 2 + cylinder_radius} 0 ${link_height / 2}"/>
+            <geometry>
+                <box size="${link_length} ${link_width} ${link_height}"/>
+            </geometry>
+        </collision>
     </link>
-    <joint name="joint0" type="continuous">
-        <parent link="link0"/>
+    <joint name="joint0" type="fixed">
+        <parent link="world"/>
         <child link="link1"/>
+    </joint>
+    <joint name="joint1" type="continuous">
+        <limit effort="30" velocity="1.0"/>
+        <parent link="link1"/>
+        <child link="link2"/>
         <origin xyz="0 0 0" rpy="0 0 0"/>
         <axis xyz="0 0 1"/>
     </joint>
-    <joint name="joint1" type="continuous">
-        <parent link="link1"/>
-        <child link="link2"/>
+    <joint name="joint2" type="continuous">
+        <limit effort="30" velocity="1.0"/>
+        <parent link="link2"/>
+        <child link="link3"/>
         <origin xyz="${link_length} 0 ${link_height}" rpy="0 0 0"/>
         <axis xyz="0 0 1"/>
     </joint>
+    <joint name="joint3" type="fixed">
+        <parent link="link3"/>
+        <child link="link4"/>
+        <origin xyz="0 0 0" rpy="0 0 0"/>
+    </joint>
 </robot>

Commit message: Adding build changes, launch file changes, and new main.rs and gpio.rs to board_arm_control

File: src/simulation/urdf/board_arm.urdf.xacro (robot description, xacro)
@@ -1,10 +1,13 @@
 <?xml version="1.1"?>
+<!-- tutorial for gazebo & URDF integration:
+https://classic.gazebosim.org/tutorials?tut=ros_urdf -->
 <robot xmlns:xacro="http://www.ros.org/wiki/xacro" name="board_arm">
+    <xacro:arg name="link_length" default="0.2"/>
     <xacro:property name="tile_size" value="0.25"/>
-    <xacro:property name="link_length" value="${tile_size * 5 * sqrt(2) / 2 - cylinder_radius}"/>
+    <xacro:property name="link_mass" value="0.1"/>
+    <xacro:property name="link_height" value="0.1"/>
     <xacro:property name="link_width" value="0.1"/>
-    <xacro:property name="link_height" value="0.1"/>
     <xacro:property name="cylinder_radius" value="${link_width / 2}"/>
-    <xacro:property name="link_mass" value="0.1"/>
+    <xacro:property name="link_length" value="$(arg link_length)"/>
     <gazebo>
         <plugin name="gazebo_ros_control" filename="libgazebo_ros_control.so">

Commit message: now able to programmatically send control commands to simulation

File: src/simulation/urdf/board_arm.urdf.xacro (robot description, xacro)
@@ -4,5 +4,5 @@
 <robot xmlns:xacro="http://www.ros.org/wiki/xacro" name="board_arm">
     <xacro:arg name="link_length" default="0.2"/>
-    <xacro:property name="tile_size" value="0.25"/>
+    <xacro:arg name="tile_size" default="0.25"/>
     <xacro:property name="link_mass" value="0.1"/>
     <xacro:property name="link_height" value="0.1"/>
@@ -10,4 +10,5 @@
     <xacro:property name="cylinder_radius" value="${link_width / 2}"/>
     <xacro:property name="link_length" value="$(arg link_length)"/>
+    <xacro:property name="tile_size" value="$(arg tile_size)"/>
     <gazebo>
         <plugin name="gazebo_ros_control" filename="libgazebo_ros_control.so">
